File: MCU Datalogger.kicad_sch (KiCad schematic)
At the start: 2 parts

Commit message: Add files via upload
Parts:
- added R3, R4, R5, R6, R7, R8: 300, symbol Device:R
Changed lines of the file:
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@@
     (rev "1")
   )
+  (symbol (lib_id "Device:R") (at 100.33 82.55 0) (unit 1)
+    (in_bom yes) (on_board yes) (dnp no) (fields_autoplaced)
+    (property "Reference" "R4" (at 102.87 81.28 0)
+      (effects (font (size 1.27 1.27)) (justify left))
+    )
+    (property "Value" "300" (at 102.87 83.82 0)
+      (effects (font (size 1.27 1.27)) (justify left))
+    )
+    (property "Footprint" "" (at 98.552 82.55 90)
+      (effects (font (size 1.27 1.27)) hide)
+    )
+    (property "Datasheet" "~" (at 100.33 82.55 0)
+      (effects (font (size 1.27 1.27)) hide)
+    )
+    (property "Purpose" "" (at 100.33 82.55 0)
+      (effects (font (size 1.27 1.27)) hide)
+    )
+    (pin "2")
+    (pin "1")
+    (instances
+      (project "MCU Datalogger"
+        (path "/6c77a3d9-2ce1-42b9-b7bb-c307dd6267ca"
+          (reference "R4") (unit 1)
+        )
+      )
+    )
+  )
   (symbol (lib_id "Device:R") (at 149.86 72.39 0) (unit 1)
     (in_bom yes) (on_board yes) (dnp no) (fields_autoplaced)
@@
     )
   )
+  (symbol (lib_id "Device:R") (at 72.39 82.55 0) (unit 1)
+    (in_bom yes) (on_board yes) (dnp no) (fields_autoplaced)
+    (property "Reference" "R3" (at 74.93 81.28 0)
+      (effects (font (size 1.27 1.27)) (justify left))
+    )
+    (property "Value" "300" (at 74.93 83.82 0)
+      (effects (font (size 1.27 1.27)) (justify left))
+    )
+    (property "Footprint" "" (at 70.612 82.55 90)
+      (effects (font (size 1.27 1.27)) hide)
+    )
+    (property "Datasheet" "~" (at 72.39 82.55 0)
+      (effects (font (size 1.27 1.27)) hide)
+    )
+    (property "Purpose" "" (at 72.39 82.55 0)
+      (effects (font (size 1.27 1.27)) hide)
+    )
+    (pin "2")
+    (pin "1")
+    (instances
+      (project "MCU Datalogger"
+        (path "/6c77a3d9-2ce1-42b9-b7bb-c307dd6267ca"
+          (reference "R3") (unit 1)
+        )
+      )
+    )
+  )
+  (symbol (lib_id "Device:R") (at 212.09 95.25 0) (unit 1)
+    (in_bom yes) (on_board yes) (dnp no) (fields_autoplaced)
+    (property "Reference" "R8" (at 214.63 93.98 0)
+      (effects (font (size 1.27 1.27)) (justify left))
+    )
+    (property "Value" "300" (at 214.63 96.52 0)
+      (effects (font (size 1.27 1.27)) (justify left))
+    )
+    (property "Footprint" "" (at 210.312 95.25 90)
+      (effects (font (size 1.27 1.27)) hide)
+    )
+    (property "Datasheet" "~" (at 212.09 95.25 0)
+      (effects (font (size 1.27 1.27)) hide)
+    )
+    (property "Purpose" "" (at 212.09 95.25 0)
+      (effects (font (size 1.27 1.27)) hide)
+    )
+    (pin "2")
+    (pin "1")
+    (instances
+      (project "MCU Datalogger"
+        (path "/6c77a3d9-2ce1-42b9-b7bb-c307dd6267ca"
+          (reference "R8") (unit 1)
+        )
+      )
+    )
+  )
+  (symbol (lib_id "Device:R") (at 134.62 105.41 0) (unit 1)
+    (in_bom yes) (on_board yes) (dnp no) (fields_autoplaced)
+    (property "Reference" "R5" (at 137.16 104.14 0)
+      (effects (font (size 1.27 1.27)) (justify left))
+    )
+    (property "Value" "300" (at 137.16 106.68 0)
+      (effects (font (size 1.27 1.27)) (justify left))
+    )
+    (property "Footprint" "" (at 132.842 105.41 90)
+      (effects (font (size 1.27 1.27)) hide)
+    )
+    (property "Datasheet" "~" (at 134.62 105.41 0)
+      (effects (font (size 1.27 1.27)) hide)
+    )
+    (property "Purpose" "" (at 134.62 105.41 0)
+      (effects (font (size 1.27 1.27)) hide)
+    )
+    (pin "2")
+    (pin "1")
+    (instances
+      (project "MCU Datalogger"
+        (path "/6c77a3d9-2ce1-42b9-b7bb-c307dd6267ca"
+          (reference "R5") (unit 1)
+        )
+      )
+    )
+  )
   (symbol (lib_id "Device:R") (at 121.92 72.39 0) (unit 1)
     (in_bom yes) (on_board yes) (dnp no) (fields_autoplaced)
@@
         )
       )
+    )
+  )
+  (symbol (lib_id "Device:R") (at 184.15 95.25 0) (unit 1)
+    (in_bom yes) (on_board yes) (dnp no) (fields_autoplaced)
+    (property "Reference" "R7" (at 186.69 93.98 0)
+      (effects (font (size 1.27 1.27)) (justify left))
+    )
+    (property "Value" "300" (at 186.69 96.52 0)
+      (effects (font (size 1.27 1.27)) (justify left))
+    )
+    (property "Footprint" "" (at 182.372 95.25 90)
+      (effects (font (size 1.27 1.27)) hide)
+    )
+    (property "Datasheet" "~" (at 184.15 95.25 0)
+      (effects (font (size 1.27 1.27)) hide)
+    )
+    (property "Purpose" "" (at 184.15 95.25 0)
+      (effects (font (size 1.27 1.27)) hide)
+    )
+    (pin "2")
+    (pin "1")
+    (instances
+      (project "MCU Datalogger"
+        (path "/6c77a3d9-2ce1-42b9-b7bb-c307dd6267ca"
+          (reference "R7") (unit 1)
+        )
+      )
+    )
+  )
+  (symbol (lib_id "Device:R") (at 162.56 105.41 0) (unit 1)
+    (in_bom yes) (on_board yes) (dnp no) (fields_autoplaced)
+    (property "Reference" "R6" (at 165.1 104.14 0)
+      (effects (font (size 1.27 1.27)) (justify left))
+    )
+    (property "Value" "300" (at 165.1 106.68 0)
+      (effects (font (size 1.27 1.27)) (justify left))
+    )
+    (property "Footprint" "" (at 160.782 105.41 90)
+      (effects (font (size 1.27 1.27)) hide)
+    )
+    (property "Datasheet" "~" (at 162.56 105.41 0)
+      (effects (font (size 1.27 1.27)) hide)
+    )
+    (property "Purpose" "" (at 162.56 105.41 0)
+      (effects (font (size 1.27 1.27)) hide)
+    )
+    (pin "2")
+    (pin "1")
+    (instances
+      (project "MCU Datalogger"
+        (path "/6c77a3d9-2ce1-42b9-b7bb-c307dd6267ca"
+          (reference "R6") (unit 1)
+        )
+      )
